Commit message: File Misplacement Fixed

File: urdf/car.urdf.xacro (robot description, xacro)
@@ -1,5 +1,17 @@
 <?xml version="1.0"?>
 <robot name="simple_car" xmlns:xacro="http://ros.org/wiki/xacro">
-  <!-- Base -->
+  <!-- ===================== -->
+  <!-- Materials (optional) -->
+  <!-- ===================== -->
+  <material name="blue">
+    <color rgba="0 0 1 1"/>
+  </material>
+  <!-- ===================== -->
+  <!-- Dummy root link       -->
+  <!-- ===================== -->
+  <link name="base_footprint"/>
+  <!-- ===================== -->
+  <!-- Base link             -->
+  <!-- ===================== -->
   <link name="base_link">
     <visual>
@@ -7,7 +19,5 @@
         <box size="0.6 0.3 0.15"/>
       </geometry>
-      <material name="blue">
-      	<color rgba="0 0 1 1"/>
-      </material>
+      <material name="blue"/>
     </visual>
     <collision>
@@ -17,12 +27,21 @@
     </collision>
     <inertial>
+      <origin xyz="0 0 0"/>
       <mass value="10.0"/>
-      <origin xyz="0 0 0"/>
-      <inertia ixx="1" ixy="0" ixz="0"
-               iyy="1" iyz="0"
-               izz="1"/>
+      <inertia
+        ixx="1.0" ixy="0.0" ixz="0.0"
+        iyy="1.0" iyz="0.0"
+        izz="1.0"/>
     </inertial>
   </link>
-  <!-- Left wheel -->
+  <!-- base_footprint → base_link -->
+  <joint name="base_footprint_joint" type="fixed">
+    <parent link="base_footprint"/>
+    <child link="base_link"/>
+    <origin xyz="0 0 0"/>
+  </joint>
+  <!-- ===================== -->
+  <!-- Wheels                -->
+  <!-- ===================== -->
   <link name="left_wheel">
     <visual>
@@ -31,6 +50,17 @@
       </geometry>
     </visual>
+    <collision>
+      <geometry>
+        <cylinder radius="0.08" length="0.05"/>
+      </geometry>
+    </collision>
+    <inertial>
+      <mass value="1.0"/>
+      <inertia
+        ixx="0.01" ixy="0.0" ixz="0.0"
+        iyy="0.01" iyz="0.0"
+        izz="0.01"/>
+    </inertial>
   </link>
-  <!-- Right wheel -->
   <link name="right_wheel">
     <visual>
@@ -39,4 +69,16 @@
       </geometry>
     </visual>
+    <collision>
+      <geometry>
+        <cylinder radius="0.08" length="0.05"/>
+      </geometry>
+    </collision>
+    <inertial>
+      <mass value="1.0"/>
+      <inertia
+        ixx="0.01" ixy="0.0" ixz="0.0"
+        iyy="0.01" iyz="0.0"
+        izz="0.01"/>
+    </inertial>
   </link>
   <!-- Wheel joints -->
@@ -53,5 +95,7 @@
     <axis xyz="0 1 0"/>
   </joint>
-  <!-- LiDAR -->
+  <!-- ===================== -->
+  <!-- LiDAR                 -->
+  <!-- ===================== -->
   <link name="lidar_link">
     <visual>
@@ -66,5 +110,8 @@
     <origin xyz="0.2 0 0.1"/>
   </joint>
-  <!-- Gazebo plugins -->
+  <!-- ===================== -->
+  <!-- Gazebo plugins        -->
+  <!-- ===================== -->
+  <!-- Differential drive -->
   <gazebo>
     <plugin name="diff_drive" filename="libgazebo_ros_diff_drive.so">
@@ -74,12 +121,13 @@
       <left_joint>left_wheel_joint</left_joint>
       <right_joint>right_wheel_joint</right_joint>
-      <wheel_separation>0.3</wheel_separation>
+      <wheel_separation>0.30</wheel_separation>
       <wheel_radius>0.08</wheel_radius>
       <cmd_vel_topic>cmd_vel</cmd_vel_topic>
       <odom_topic>odom</odom_topic>
       <publish_tf>true</publish_tf>
-      <robot_base_frame>base_link</robot_base_frame>
+      <robot_base_frame>base_footprint</robot_base_frame>
     </plugin>
   </gazebo>
+  <!-- 2D LiDAR -->
   <gazebo reference="lidar_link">
     <sensor name="lidar" type="ray">
@@ -101,4 +149,5 @@
         <topicName>scan</topicName>
         <frameName>lidar_link</frameName>
+        <output_type>sensor_msgs/LaserScan</output_type>
       </plugin>
     </sensor>
